File: leds.kicad_sch (KiCad schematic)
At the start: 15 parts, among them Q8 YJQ3400A-YAN, Q9 YJQ3400A-YAN

Commit message: Board routed
Parts:
- removed J_REAR_LAMP: Conn_01x02, symbol Connector_Generic:Conn_01x02
- Q8, Q9: footprint Package_DFN_QFN:Diodes_UDFN2020-6_Type-F -> footprints:DFN2020-6L
Connections:
- net REAR_LEDS_K: now reaches R16.1
- net V_LEDS renamed REAR_LEDS_A
Changed lines of the file:
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@@
     (effects (font (size 1.27 1.27)) (justify left))
+  )
+  (hierarchical_label "REAR_LEDS_A" (shape output) (at 127 55.88 180) (fields_autoplaced)
+    (effects (font (size 1.27 1.27)) (justify right))
   )
   (hierarchical_label "LED1_GATE" (shape input) (at 236.22 74.93 0) (fields_autoplaced)
@@
     (effects (font (size 1.27 1.27)) (justify left))
   )
+  (hierarchical_label "REAR_LEDS_K" (shape input) (at 127 58.42 180) (fields_autoplaced)
+    (effects (font (size 1.27 1.27)) (justify right))
+  )
   (hierarchical_label "V_LEDS" (shape input) (at 198.12 45.72 0) (fields_autoplaced)
     (effects (font (size 1.27 1.27)) (justify left))
@@
       (effects (font (size 1.27 1.27)) (justify left))
     )
-    (property "Footprint" "Package_DFN_QFN:Diodes_UDFN2020-6_Type-F" (at 148.59 96.52 0)
+    (property "Footprint" "footprints:DFN2020-6L" (at 148.59 96.52 0)
       (effects (font (size 1.27 1.27)) hide)
     )
@@
       (effects (font (size 1.27 1.27)) (justify left))
     )
-    (property "Footprint" "Package_DFN_QFN:Diodes_UDFN2020-6_Type-F" (at 190.5 74.93 0)
+    (property "Footprint" "footprints:DFN2020-6L" (at 190.5 74.93 0)
       (effects (font (size 1.27 1.27)) hide)
     )
@@
       (effects (font (size 1.27 1.27)) (justify left))
     )
-    (property "Footprint" "Package_DFN_QFN:Diodes_UDFN2020-6_Type-F" (at 168.91 82.55 0)
+    (property "Footprint" "footprints:DFN2020-6L" (at 168.91 82.55 0)
       (effects (font (size 1.27 1.27)) hide)
     )
@@
     )
   )
-  (symbol (lib_id "Connector_Generic:Conn_01x02") (at 121.92 58.42 180) (unit 1)
-    (in_bom yes) (on_board yes) (dnp no)
-    (property "Reference" "J_REAR_LAMP" (at 121.92 50.8 0)
-      (effects (font (size 1.27 1.27)))
-    )
-    (property "Value" "Conn_01x02" (at 121.92 53.34 0)
-      (effects (font (size 1.27 1.27)))
-    )
-    (property "Footprint" "" (at 121.92 58.42 0)
-      (effects (font (size 1.27 1.27)) hide)
-    )
-    (property "Datasheet" "~" (at 121.92 58.42 0)
-      (effects (font (size 1.27 1.27)) hide)
-    )
-    (pin "1")
-    (pin "2")
-    (instances
-      (project "bikelamp"
-        (path "/fa1ac838-ddbb-4559-ade6-578710b3e6ec"
-          (reference "J_REAR_LAMP") (unit 1)
-        )
-        (path "/fa1ac838-ddbb-4559-ade6-578710b3e6ec/a1559bb5-2c5f-4b98-ad82-ef9f27fe5cb2"
-          (reference "J_REAR_LAMP1") (unit 1)
-        )
-      )
-    )
-  )
   (symbol (lib_id "Device:R_Small") (at 193.04 64.77 0) (unit 1)
     (in_bom yes) (on_board yes) (dnp no) (fields_autoplaced)
@@
       (effects (font (size 1.27 1.27)) (justify left))
     )
-    (property "Footprint" "Package_DFN_QFN:Diodes_UDFN2020-6_Type-F" (at 128.27 111.76 0)
-      (effects (font (size 1.27 1.27)) hide)
-    )
+    (property "Footprint" "footprints:DFN2020-6L" (at 128.27 111.76 0)
+      (effects (font (size 1.27 1.27)) hide)
+    )

Commit message: - Get rid from <0.3 mm drills - Fine tune GND fill
Connections:
- net REAR_LEDS_A renamed V_LEDS
Changed lines of the file:
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@@
   (junction (at 193.04 45.72) (diameter 0) (color 0 0 0 0)
-  )
-  (junction (at 151.13 45.72) (diameter 0) (color 0 0 0 0)
   )
   (junction (at 151.13 121.92) (diameter 0) (color 0 0 0 0)
@@
   )
   (wire (pts (xy 179.07 82.55) (xy 222.25 82.55))
-    (stroke (width 0) (type default))
-  )
-  (wire (pts (xy 127 55.88) (xy 130.81 55.88))
     (stroke (width 0) (type default))
   )
@@
     (stroke (width 0) (type default))
   )
-  (wire (pts (xy 130.81 55.88) (xy 130.81 45.72))
-    (stroke (width 0) (type default))
-  )
   (wire (pts (xy 171.45 59.69) (xy 171.45 62.23))
     (stroke (width 0) (type default))
@@
   )
   (wire (pts (xy 130.81 121.92) (xy 130.81 123.19))
-    (stroke (width 0) (type default))
-  )
-  (wire (pts (xy 130.81 45.72) (xy 151.13 45.72))
     (stroke (width 0) (type default))
   )
@@
     (effects (font (size 1.27 1.27)) (justify left))
   )
-  (hierarchical_label "REAR_LEDS_A" (shape output) (at 127 55.88 180) (fields_autoplaced)
-    (effects (font (size 1.27 1.27)) (justify right))
-  )
   (hierarchical_label "LED1_GATE" (shape input) (at 236.22 74.93 0) (fields_autoplaced)
